Commit message: Update 2r robot urdf

File: src/02_robot_description/urdf/two_r_robot.urdf (robot description, URDF)
Before this commit: robot 2R_robot, 3 links, 2 joints
Joints:
- joint joint_1: axis 0 1 0 -> 0 0 1
- joint joint_2: axis 0 1 0 -> 0 0 1; origin xyz=0 0 1.0 rpy=0 0 0 -> xyz=1.0 0 0 rpy=0 0 0
