Commit message: Add lecture7 moveit config

File: src/02_robot_description/urdf/rrbot.urdf (robot description, URDF)
Before this commit: robot 2R_robot, 3 links, 2 joints
Joints:
- joint joint_1: axis 0 0 1 -> 0 1 0; limit lower=-3.14159 upper=3.14159 effort=10 velocity=1 -> lower=-1.5 upper=1.5 effort=10 velocity=1
- joint joint_2: axis 0 0 1 -> 0 1 0; origin xyz=1.0 0 0 rpy=0 0 0 -> xyz=0 0 1.0 rpy=0 0 0
